File: schematics/PIC12F_boost_2021_09_29_A.sch (EAGLE design)
At the start: 29 parts, among them IC1 PIC12F510/SN, Q1 FMMT491ATA, Q2 FMMT591A, Q3 FDT457N

Commit message: Add files via upload
Parts:
- IC1: value PIC12F510/SN -> PIC12F1501
Other:
- note added: "6/24/2022 Updated PIC to correct part number"
Changed lines of the file:
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@@
 <setting verticaltext="up"/>
 </settings>
-<grid distance="50" unitdist="mil" unit="mil" style="lines" multiple="1" display="yes" altdistance="0.01" altunitdist="inch" altunit="inch"/>
+<grid distance="0.1" unitdist="inch" unit="inch" style="lines" multiple="1" display="no" altdistance="0.01" altunitdist="inch" altunit="inch"/>
 <layers>
 <layer number="1" name="Top" color="4" fill="1" visible="no" active="no"/>
@@
 </classes>
 <parts>
-<part name="IC1" library="microchip_pic12f" deviceset="PIC12F510" device="/SN"/>
+<part name="IC1" library="microchip_pic12f" deviceset="PIC12F510" device="/SN" value="PIC12F1501"/>
 <part name="Q1" library="SparkFun-DiscreteSemi" deviceset="TRANSISTOR_NPN" device="MMBT5088" value="FMMT491ATA"/>
 <part name="Q2" library="SparkFun-DiscreteSemi" deviceset="TRANSISTOR_PNP" device="MMBT4403" value="FMMT591A"/>
@@
 Solder This Jumper for current mode.
 Do not populate R5,R6 or R8 if jumper is made.</text>
+<text x="111.76" y="58.42" size="1.778" layer="97">6/24/2022
+Updated PIC to correct part number</text>
 </plain>
 <instances>
