File: schematics/PIC12F_boost_2021_09_29_A.brd (EAGLE design)
At the start: 45.4 x 38.7 mm, 29 parts, among them IC1 PIC12F510/SN, Q1 FMMT491ATA, Q2 FMMT591A, Q3 FDT457N

Commit message: Add files via upload
Parts:
- IC1: value PIC12F510/SN -> PIC12F1501
Changed lines of the file:
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@@
 <attribute name="NAME" x="56.642" y="13.97" size="0.4064" layer="25" rot="R90"/>
 </element>
-<element name="IC1" library="microchip_pic12f" package="SOIC8-SN" value="PIC12F510/SN" x="43.18" y="16.51" smashed="yes" rot="R270">
+<element name="IC1" library="microchip_pic12f" package="SOIC8-SN" value="PIC12F1501" x="43.18" y="16.51" smashed="yes" rot="R270">
 <attribute name="NAME" x="45.67" y="19.327" size="0.8128" layer="25"/>
 </element>
